File: Blimp/OpenMV Breakout Board/OpenMV Breakout Board.kicad_pcb (KiCad board)
At the start: 2 copper layers, 35.6 x 26.7 mm, 20 parts, among them J1 UART3, J2 Detector, J3 Servo, J4 Debug, M1 OPENMV3, U1 ATWINC1500, U2 74LVC1G17

Commit message: Updates to OpenMV hat to make pin labels more legible on PCB. Change schematic to be A paper sized for printing, reorg for readability
Connections:
- net /P7 renamed /Servo2_PWM
Other:
- board text added: "3V3 ~ G"
- board text added: "5V TX RX G"
- board text added: "5V ~ G"
- board text added: "Detector"
- board text added: "GND"
- board text added: "J1"
- board text added: "RX"
- board text added: "Servos"
- board text added: "TX"
Changed lines of the file:
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@@
   (net 11 "/DBG_TX")
   (net 12 "/DBG_RX")
-  (net 13 "/P7")
+  (net 13 "/Servo2_PWM")
   (net 14 "Net-(R3-Pad2)")
   (net 15 "Net-(R4-Pad1)")
@@
       (net 1 "+5V") (pinfunction "Pin_1") (pintype "passive"))
     (pad "2" thru_hole oval (at 0 2.54 270) (size 1.7 1.7) (drill 1) (layers *.Cu *.Mask)
-      (net 13 "/P7") (pinfunction "Pin_2") (pintype "passive"))
+      (net 13 "/Servo2_PWM") (pinfunction "Pin_2") (pintype "passive"))
     (pad "3" thru_hole oval (at 0 5.08 270) (size 1.7 1.7) (drill 1) (layers *.Cu *.Mask)
       (net 8 "GND") (pinfunction "Pin_3") (pintype "passive"))
@@
       (net 1 "+5V") (pinfunction "VIN") (pintype "power_out"))
     (pad "11" thru_hole circle (at 33.909 -6.604) (size 1.778 1.778) (drill 1.016) (layers *.Cu *.Paste *.Mask)
-      (net 13 "/P7") (pinfunction "P7") (pintype "bidirectional"))
+      (net 13 "/Servo2_PWM") (pinfunction "P7") (pintype "bidirectional"))
     (pad "12" thru_hole circle (at 33.909 -9.144) (size 1.778 1.778) (drill 1.016) (layers *.Cu *.Paste *.Mask)
       (net 20 "/IRQ") (pinfunction "P8") (pintype "bidirectional"))
@@
       (net 18 "/Mod_RST") (pinfunction "C") (pintype "passive"))
     (pad "3" smd custom (at 1.3 0 90) (size 1 0.5) (layers "F.Cu" "F.Mask")
-      (net 13 "/P7") (pinfunction "B") (pintype "passive") (zone_connect 2)
+      (net 13 "/Servo2_PWM") (pinfunction "B") (pintype "passive") (zone_connect 2)
       (options (clearance outline) (anchor rect))
       (primitives
@@
     (property "Sheetname" "")
     (attr smd)
-    (fp_text reference "C3" (at 2.667 0.127 90) (layer "B.SilkS")
+    (fp_text reference "C3" (at 2.413 -1.016 90) (layer "B.SilkS")
       (effects (font (size 1 1) (thickness 0.15)) (justify mirror))
     )
@@
     (property "Sheetname" "")
     (attr smd)
-    (fp_text reference "R4" (at 0 1.43 90) (layer "B.SilkS")
+    (fp_text reference "R4" (at 2.667 0 90) (layer "B.SilkS")
       (effects (font (size 1 1) (thickness 0.15)) (justify mirror))
     )
@@
     (property "Sheetname" "")
     (attr smd)
-    (fp_text reference "C7" (at -2.667 0 90) (layer "B.SilkS")
+    (fp_text reference "C7" (at 0.635 -1.27 90) (layer "B.SilkS")
       (effects (font (size 1 1) (thickness 0.15)) (justify mirror))
     )
@@
     (property "Sheetname" "")
     (attr smd)
-    (fp_text reference "C5" (at -2.794 0 90) (layer "B.SilkS")
+    (fp_text reference "C5" (at 2.794 0 90) (layer "B.SilkS")
       (effects (font (size 1 1) (thickness 0.15)) (justify mirror))
     )
@@
     (property "Sheetname" "")
     (attr smd)
-    (fp_text reference "C1" (at 0 1.85 90) (layer "B.SilkS")
+    (fp_text reference "C1" (at 2.921 1.016 90) (layer "B.SilkS")
       (effects (font (size 1 1) (thickness 0.15)) (justify mirror))
     )
@@
     (property "Sheetname" "")
     (attr smd)
-    (fp_text reference "C6" (at -2.667 0 90) (layer "B.SilkS")
+    (fp_text reference "C6" (at 2.6405 0 90) (layer "B.SilkS")
       (effects (font (size 1 1) (thickness 0.15)) (justify mirror))
     )
@@
     (effects (font (size 1.016 1.016) (thickness 0.127)) (justify mirror))
   )
+  (gr_text "Detector" (at 135.763 113.157) (layer "B.SilkS")
+    (effects (font (size 0.889 0.9652) (thickness 0.15)) (justify mirror))
+  )
+  (gr_text "RX" (at 124.079 104.267) (layer "B.SilkS")
+    (effects (font (size 0.889 0.9652) (thickness 0.15)) (justify mirror))
+  )
+  (gr_text "GND" (at 124.333 106.807) (layer "B.SilkS")
+    (effects (font (size 0.889 0.9652) (thickness 0.15)) (justify mirror))
+  )
+  (gr_text "3V3 ~  G" (at 136.271 114.554) (layer "B.SilkS")
+    (effects (font (size 0.889 0.9652) (thickness 0.15)) (justify mirror))
+  )
+  (gr_text "5V TX RX  G" (at 126.111 115.189) (layer "B.SilkS")
+    (effects (font (size 0.889 0.9652) (thickness 0.15)) (justify mirror))
+  )
+  (gr_text "J1" (at 129.54 113.665) (layer "B.SilkS")
+    (effects (font (size 0.889 0.9652) (thickness 0.15)) (justify mirror))
+  )
+  (gr_text "Servos" (at 145.288 110.871) (layer "B.SilkS")
+    (effects (font (size 0.889 0.9652) (thickness 0.15)) (justify mirror))
+  )
+  (gr_text "5V  ~  G" (at 145.034 112.141) (layer "B.SilkS")
+    (effects (font (size 0.889 0.9652) (thickness 0.15)) (justify mirror))
+  )
+  (gr_text "TX" (at 124.079 101.981) (layer "B.SilkS")
+    (effects (font (size 0.889 0.9652) (thickness 0.15)) (justify mirror))
+  )
   (gr_text "TMR|P7" (at 145.796 109.601 90) (layer "F.SilkS")
     (effects (font (size 0.762 0.762) (thickness 0.15)))
@@
     (effects (font (size 0.889 0.9652) (thickness 0.15)))
   )
+  (gr_text "TX" (at 123.698 99.822 90) (layer "F.SilkS")
+    (effects (font (size 0.889 0.9652) (thickness 0.15)))
+  )
   (gr_text "G   ~ 3V3" (at 135.89 114.935) (layer "F.SilkS")
     (effects (font (size 0.889 0.9652) (thickness 0.15)))
   )
+  (gr_text "RX" (at 123.825 104.14 90) (layer "F.SilkS")
+    (effects (font (size 0.889 0.9652) (thickness 0.15)))
+  )
   (gr_text "RST Sel" (at 142.367 108.712 90) (layer "F.SilkS")
     (effects (font (size 1 1) (thickness 0.15)))
   )
+  (gr_text "GND" (at 121.793 108.712) (layer "F.SilkS")
+    (effects (font (size 0.889 0.9652) (thickness 0.15)))
+  )
   (gr_text "G  RX TX 5V" (at 125.857 114.935) (layer "F.SilkS")

Commit message: additional labels on pcb for servos
Other:
- board text added: "5V P7 G 5V P9 G"
- board text removed: "5V ~ G"
Changed lines of the file:
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@@
     (effects (font (size 0.889 0.9652) (thickness 0.15)) (justify mirror))
   )
-  (gr_text "Servos" (at 145.288 110.871) (layer "B.SilkS")
+  (gr_text "Servos" (at 145.288 109.474) (layer "B.SilkS")
     (effects (font (size 0.889 0.9652) (thickness 0.15)) (justify mirror))
   )
-  (gr_text "5V  ~  G" (at 145.034 112.141) (layer "B.SilkS")
+  (gr_text "5V P7  G\n5V P9  G" (at 144.907 111.633) (layer "B.SilkS")
     (effects (font (size 0.889 0.9652) (thickness 0.15)) (justify mirror))
   )
